Commit message: joints complete

File: three_link.urdf (robot description, URDF)
Before this commit: robot robot, 3 links, 2 joints
Joints:
- joint Torso_BackLeg: origin xyz=1.0 1.0 0.5 rpy=0 0 0 -> xyz=1.0 0.0 0.5 rpy=0 0 0
- joint Torso_FrontLeg: origin xyz=2.0 1.0 0.5 rpy=0 0 0 -> xyz=2.0 0.0 0.5 rpy=0 0 0
